Commit message: Update Arm.xacro

File: Arm/Arm/Arm_description/urdf/Arm.xacro (robot description, xacro)
@@ -94,5 +94,5 @@
   <parent link="Lengan1_1"/>
   <child link="Lengan2_1"/>
-  <axis xyz="1.0 -0.0 -0.0"/>
+  <axis xyz="-1.0 -0.0 -0.0"/>
 </joint>
 <joint name="Revolute 3" type="continuous">
